File: hpdl_1414_pmod.kicad_pcb (KiCad board)
At the start: 2 copper layers, 84 x 56 mm, 15 parts, among them J1 10129382-912001BLF, J2 10129382-912001BLF

Commit message: Update schematics
Parts:
- removed C3: CP, Capacitor_THT:C_Disc_D4.3mm_W1.9mm_P5.00mm
- removed C4: 15uF, Capacitor_SMD:C_1210_3225Metric_Pad1.33x2.70mm_HandSolder
- moved C2 40.8 mm to (107.5, 73.5), turned to 180 degrees
- moved C1 25.8 mm to (107.5, 70.5), turned to 180 degrees
Connections:
- J2 pad 11: GND -> unconnected-(J2-GND-Pad11)
- J2 pad 12: VDD -> unconnected-(J2-VCC-Pad12)
- J2 pad 5: GND -> unconnected-(J2-GND-Pad5)
- J2 pad 6: VDD -> unconnected-(J2-VCC-Pad6)
Routing:
- net VDD: track 167.9 -> 117.6 mm
- net GND: track 11.7 -> 0.00 mm
